Commit message: refresh

File: src/bioloid_gp_description/bioloid_gp4/urdf/bioloid_gp4.urdf (robot description, URDF)
Before this commit: robot bioloid_gp4, 22 links, 21 joints
Joints:
- joint joint_1: origin xyz=0.00874999999999919 -0.0564904194241639 0.00275000000000068 rpy=3.14159265358979 0 3.14159265358979 -> xyz=0.00874999999999919 -0.0564904194241639 0.00275000000000068 rpy=3.14159265358979 0 0
- joint joint_10: origin xyz=0.016 -0.0535000000000007 0 rpy=3.14159265358979 0 -3.14159265358979 -> xyz=0.016 -0.0535000000000007 0 rpy=3.14159265358979 0 3.14159265358979
- joint joint_13: origin xyz=0 -0.0744000000000003 -0.0145000000000005 rpy=0 0 3.14159265358979 -> xyz=0 -0.0744000000000003 0.0145000000000005 rpy=0 0 3.14159265358979
- joint joint_15: origin xyz=0 0.0750000000000001 0.0145 rpy=-1.5707963267949 0 3.14159265358979 -> xyz=0 0.0750000000000001 -0.0145 rpy=-1.5707963267949 0 3.14159265358979
- joint joint_17: origin xyz=-0.0138000000000001 0 -9.99999999998225E-05 rpy=1.5707963267949 0 -1.5707963267949 -> xyz=0.0138000000000001 0 -9.99999999998225E-05 rpy=1.5707963267949 0 1.5707963267949
- joint joint_18: origin xyz=0.0137999999999867 0 -9.9999999999989E-05 rpy=-1.5707963267949 0 1.5707963267949 -> xyz=0.0137999999999867 0 -9.9999999999989E-05 rpy=1.5707963267949 0 -1.5707963267949
- joint joint_2: origin xyz=0.00874999999999918 0.0564904194241643 0.00275 rpy=3.14159265358979 0 0 -> xyz=0.00874999999999918 0.0564904194241643 0.00275 rpy=3.14159265358979 0 3.1416
- joint joint_20: origin xyz=0.00025 0 0.05555 rpy=3.1416 0 -1.5708 -> xyz=0.00025 0 0.05555 rpy=3.1416 3.1416 1.5708
- joint joint_21: origin xyz=0 0 -0.0537001030776406 rpy=0 1.5707963267949 0 -> xyz=0 0 0.0537001030776406 rpy=0 -1.5707963267949 0
- joint joint_3: origin xyz=0 -0.0230095805758343 0.0179999999999891 rpy=-1.5707963267949 0 1.5707963267949 -> xyz=0 0.0230095805758343 0.0179999999999891 rpy=-1.5707963267949 0 1.5707963267949
- joint joint_4: origin xyz=0 -0.0230095805758357 0.0179999999999895 rpy=-1.5707963267949 0 -1.5707963267949 -> xyz=0 0.0230095805758357 0.0179999999999895 rpy=-1.5707963267949 0 -1.5707963267949
- joint joint_5: origin xyz=0 -0.0574 0.0182000000000002 rpy=1.5707963267949 0 0 -> xyz=0 -0.0574 -0.0182000000000002 rpy=1.5707963267949 0 0
- joint joint_6: origin xyz=0 -0.0573999999999997 0.0182000000000009 rpy=1.5707963267949 0 0 -> xyz=0 -0.0573999999999997 -0.0182000000000009 rpy=1.5707963267949 0 3.1416
- joint joint_7: origin xyz=-0.0224999999999999 0.0425 0 rpy=1.5707963267949 -1.5707963267949 0 -> xyz=0.0224999999999999 -0.0425 0 rpy=1.5707963267949 1.5707963267949 0
- joint joint_8: origin xyz=0.0225000000000024 0.0424999999999999 0 rpy=1.5707963267949 1.5707963267949 0 -> xyz=0.0225000000000024 -0.0424999999999999 0 rpy=-1.5707963267949 -1.5707963267949 0
- joint joint_9: origin xyz=-0.016 -0.0535000000000009 0 rpy=0 0 0 -> xyz=-0.016 -0.0535000000000009 0 rpy=-3.14159265358979 0 3.14159265358979

Commit message: refresh

File: src/bioloid_gp_description/bioloid_gp4/urdf/bioloid_gp4.urdf (robot description, URDF)
Before this commit: robot bioloid_gp4, 22 links, 21 joints
Links:
- added link dummy
- added link imu_link; visual box size=0.016 0.026 0.005
Joints:
- added joint dummy_joint: type fixed, parent dummy, child base_link
- added joint imu_to_base_joint: type fixed, parent base_link, child imu_link, origin xyz=0.00824999999999999 0 -0.035 rpy=0 0 0
- joint joint_2: origin xyz=0.00874999999999918 0.0564904194241643 0.00275 rpy=3.14159265358979 0 3.1416 -> xyz=0.00874999999999918 0.0564904194241643 0.00275 rpy=3.14159265358979 0 3.14159265358979
- joint joint_20: origin xyz=0.00025 0 0.05555 rpy=3.1416 3.1416 1.5708 -> xyz=0.00025 0 0.05555 rpy=3.14159265358979 3.14159265358979 1.5708
- joint joint_6: origin xyz=0 -0.0573999999999997 -0.0182000000000009 rpy=1.5707963267949 0 3.1416 -> xyz=0 -0.0573999999999997 -0.0182000000000009 rpy=1.5707963267949 0 3.14159265358979
