Commit message: update all diferent robots configurations descriptions

File: bioloid_gp_description/bioloidgp_social_robot/urdf/bioloidgp_social_robot.urdf (robot description, URDF)
Before this commit: robot bioloidgp_social_robot, 24 links, 23 joints
Links:
- removed link torso_Link
- added link torso_link, mass 0.0150306588580906; collision mesh filename=package://bioloidgp_social_robot/meshes/torso_link.STL; visual mesh filename=package://bioloidgp_social_robot/meshes/torso_link.STL
- link base_link: mass 0.23897 -> 0.38847
- link camera: mass 0.0951615153632961 -> 0.096022
- link head_link: mass 0.0131552831434282 -> 0
- link left_arm_link_1: mass 0.00402029367652142 -> 0.0040203
- link left_arm_link_2: mass 0.086643029497245 -> 0.088364
- link left_arm_link_3: mass 0.0525573198575286 -> 0.053418
- link left_gripper: mass 0.00882433124339499 -> 0.0088243
- link left_leg_link_1: mass 0.0465444227419532 -> 0.0474050276692231
- link left_leg_link_2: mass 0.0873959659250778 -> 0.0891171757796176
- link left_leg_link_3: mass 0.00701486534628872 -> 0.00701486534628874
- link left_leg_link_4: mass 0.0856772163480854 -> 0.087398
- link left_leg_link_5: mass 0.014503230384799 -> 0.014503
- link right_arm_link_1: mass 0.00402029367652138 -> 0.0040203
- link right_arm_link_2: mass 0.0866430294972451 -> 0.088364
- link right_arm_link_3: mass 0.0525573198575286 -> 0.053418
- link right_gripper: mass 0.00882433124339025 -> 0.0088243
- link right_leg_link_1: mass 0.0465444227419532 -> 0.047405027669223
- link right_leg_link_2: mass 0.0873959659250779 -> 0.0891171757796176
- link right_leg_link_3: mass 0.00701486534628872 -> 0.00701486534628873
- link right_leg_link_4: mass 0.0856772163480855 -> 0.0873984262026251
Joints:
- joint joint_1: origin xyz=0.00874999999999919 -0.0564904194241639 0.00275000000000068 rpy=3.14159265358979 0 0 -> xyz=0.00875 -0.05649 0.00275 rpy=3.1416 0 3.1416
- joint joint_10: origin xyz=0.016 -0.0535000000000007 0 rpy=3.14159265358979 0 3.14159265358979 -> xyz=0.016 -0.0535000000000006 0 rpy=0 0 0; parent torso_Link -> torso_link
- joint joint_11: origin xyz=0 -0.0417999999999986 0 rpy=0 0 0 -> xyz=0 -0.0417999999999987 0 rpy=0 0 0
- joint joint_12: origin xyz=0 -0.0418000000000006 0 rpy=3.14159265358979 0 -3.14159265358979 -> xyz=0 -0.0418000000000007 0 rpy=3.14159265358979 0 -3.14159265358979
- joint joint_13: origin xyz=0 -0.0744000000000003 0.0145000000000005 rpy=0 0 3.14159265358979 -> xyz=0 -0.0744000000000003 -0.0144999999999987 rpy=0 0 3.14159265358979
- joint joint_14: origin xyz=0 -0.0744 -0.0145000000000106 rpy=0 0 3.14159265358979 -> xyz=0 -0.0744 0.0145000000000106 rpy=0 0 -3.14159265358979
- joint joint_15: origin xyz=0 0.0750000000000001 -0.0145 rpy=-1.5707963267949 0 3.14159265358979 -> xyz=0 0.0749999999999997 0.0145000000000012 rpy=-1.57079632679491 0 -3.14159265358979
- joint joint_16: origin xyz=0 0.075 0.0144999999999907 rpy=-1.5707963267949 0 -3.14159265358979 -> xyz=0 0.0750000000000028 -0.0144999999999764 rpy=-1.57079632679471 0 3.14159265358979
- joint joint_17: axis 1 0 0 -> 0 0 1; origin xyz=0.0138000000000001 0 -9.99999999998225E-05 rpy=1.5707963267949 0 1.5707963267949 -> xyz=-0.0138000000000002 0 -9.99999999997669E-05 rpy=1.57079632679491 0 3.1416
- joint joint_18: axis 1 0 0 -> 0 0 1; origin xyz=0.0137999999999867 0 -9.9999999999989E-05 rpy=1.5707963267949 0 -1.5707963267949 -> xyz=-0.01 0 0 rpy=1.57079632679471 0 0
- joint joint_19: child torso_Link -> torso_link; origin xyz=0.00824999999999999 0 -0.05725 rpy=1.5707963267949 0 1.5707963267949 -> xyz=0.00825 0 -0.05725 rpy=1.5708 0 1.5708
- joint joint_2: origin xyz=0.00874999999999918 0.0564904194241643 0.00275 rpy=3.14159265358979 0 3.14159265358979 -> xyz=0.00875 0.05649 0.00275 rpy=3.1416 0 0
- joint joint_20: origin xyz=0.00825000000000002 0 0.0220498969223593 rpy=3.14159265358979 3.14159265358979 1.5708 -> xyz=0.00825000000000002 0 0.0220498969223593 rpy=3.14159265358979 0 -1.60287187004926
- joint joint_21: axis 0 0 1 -> 1 0 0; origin xyz=0 0 0.0537001030776406 rpy=0 -1.5707963267949 0 -> xyz=0 0 -0.05 rpy=-1.5707963267949 3.14159265358979 3.14159265358979
- joint joint_3: origin xyz=0 0.0230095805758343 0.0179999999999891 rpy=-1.5707963267949 0 1.5707963267949 -> xyz=0 -0.02301 0.018 rpy=-1.5708 0 1.5708
- joint joint_4: axis 0 0 1 -> 0 1 0; origin xyz=0 0.0230095805758357 0.0179999999999895 rpy=-1.5707963267949 0 -1.5707963267949 -> xyz=0 -0.0230095805758357 0.0179999999999604 rpy=1.5707963267949 1.5707963267949 0
- joint joint_5: origin xyz=0 -0.0574 -0.0182000000000002 rpy=1.5707963267949 0 0 -> xyz=0 -0.0574 0.0182 rpy=1.5708 0 0
- joint joint_6: origin xyz=0 -0.0573999999999997 -0.0182000000000009 rpy=1.5707963267949 0 3.14159265358979 -> xyz=-0.0573999999999997 0.0182000000000009 0 rpy=0 1.5707963267949 0
- joint joint_7: origin xyz=0.0224999999999999 -0.0425 0 rpy=1.5707963267949 1.5707963267949 0 -> xyz=-0.0225 0.0425 0 rpy=1.5707963267949 -1.5707963267949 0
- joint joint_8: origin xyz=0.0225000000000024 -0.0424999999999999 0 rpy=-1.5707963267949 -1.5707963267949 0 -> xyz=-0.0225000000000029 0.0424999999999997 0 rpy=1.5707963267949 1.5707963267949 0
- joint joint_9: origin xyz=-0.016 -0.0535000000000009 0 rpy=-3.14159265358979 0 3.14159265358979 -> xyz=-0.016 -0.0535000000000006 0 rpy=0 0 0; parent torso_Link -> torso_link
